Commit message: ROS - connect to ROS w/ joystick input
update ELI5 readme
update TODO

File: urdf/toyota_86.urdf (robot description, URDF)
Before this commit: robot tt02, 13 links, 12 joints
Links:
- link base_link: geometry visual mesh filename=file:///home/tanmay/ros2/ros2_car_ws/meshes/tt02_base_link.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 scale=10 10 10
- link wheel_frl: geometry visual mesh filename=file:///home/tanmay/ros2/ros2_car_ws/meshes/tt02_wheel.stl scale=10 10 10
- link wheel_frr: geometry visual mesh filename=file:///home/tanmay/ros2/ros2_car_ws/meshes/tt02_wheel.stl scale=10 -10 10
- link wheel_rrl: geometry visual mesh filename=file:///home/tanmay/ros2/ros2_car_ws/meshes/tt02_wheel.stl scale=10 10 10
- link wheel_rrr: geometry visual mesh filename=file:///home/tanmay/ros2/ros2_car_ws/meshes/tt02_wheel.stl scale=10 -10 10
Joints:
- joint base_frl_joint: limit lower=-0.008 upper=0.008 effort=0 velocity=0 -> lower=-0.08 upper=0.08 effort=0 velocity=0; origin xyz=0.129382 0.067852 -0.027459 rpy=0 0 0 -> xyz=1.29382 0.67852 -0.27459 rpy=0 0 0
- joint base_frr_joint: limit lower=-0.008 upper=0.008 effort=0 velocity=0 -> lower=-0.08 upper=0.08 effort=0 velocity=0; origin xyz=0.129382 -0.067852 -0.027459 rpy=0 0 0 -> xyz=1.29382 -0.67852 -0.27459 rpy=0 0 0
- joint base_rrl_joint: limit lower=-0.008 upper=0.008 effort=0 velocity=0 -> lower=-0.08 upper=0.08 effort=0 velocity=0; origin xyz=-0.129382 0.067852 -0.027459 rpy=0 0 0 -> xyz=-1.29382 0.67852 -0.27459 rpy=0 0 0
- joint base_rrr_joint: limit lower=-0.008 upper=0.008 effort=0 velocity=0 -> lower=-0.08 upper=0.08 effort=0 velocity=0; origin xyz=-0.129382 -0.067852 -0.027459 rpy=0 0 0 -> xyz=-1.29382 -0.67852 -0.27459 rpy=0 0 0
