File: hall sensor pcb/AS5600 Breakout.kicad_pcb (KiCad board)
At the start: 2 copper layers, 30 x 10 mm, 6 parts, among them J2 Conn_01x06_Pin, U1 AS5600

Commit message: make smaller, remove holes
rebase 2
Parts:
- moved C2 0.45 mm to (67.5, 59.0)
Routing:
- net GND: track 2.51 -> 4.21 mm
Other:
- board size 30 x 10 mm -> 25 x 10 mm
Changed lines of the file:
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@@
 	(footprint "Capacitor_SMD:C_0805_2012Metric"
 		(layer "F.Cu")
-		(at 67.5 58.5 90)
+		(at 67.5 58.95 90)
 		(descr "Capacitor SMD 0805 (2012 Metric), square (rectangular) end terminal, IPC-7351 nominal, (Body size source: IPC-SM-782 page 76, https://www.pcb-3d.com/wordpress/wp-content/uploads/ipc-sm-782a_amendment_1_and_2.pdf, https://docs.google.com/spreadsheets/d/1BsfQQcO9C6DZCsRaXUlFlo91Tg2WpOkGARC1WS5S8t0/edit?usp=sharing), generated with kicad-footprint-generator")
 		(tags "capacitor")
 		(property "Reference" "C2"
-			(at -6.5 -0.5 180)
+			(at -6.05 1 180)
 			(layer "F.SilkS")
 			(effects
@@
 	)
 	(gr_arc
-		(start 91 63)
-		(mid 90.12132 65.12132)
-		(end 88 66)
+		(start 91 63.5)
+		(mid 90.267767 65.267767)
+		(end 88.5 66)
 		(stroke
 			(width 0.15)
@@
 		(layer "Edge.Cuts")
 	)
-	(gr_circle
-		(center 64 59)
-		(end 65.414 59)
+	(gr_line
+		(start 66 63)
+		(end 66 58.5)
 		(stroke
 			(width 0.15)
 			(type solid)
 		)
-		(fill no)
 		(layer "Edge.Cuts")
 	)
-	(gr_line
-		(start 61 63)
-		(end 61 59)
+	(gr_arc
+		(start 88.5 56)
+		(mid 90.267767 56.732233)
+		(end 91 58.5)
 		(stroke
 			(width 0.15)
@@
 		(layer "Edge.Cuts")
 	)
-	(gr_arc
-		(start 88 56)
-		(mid 90.12132 56.87868)
-		(end 91 59)
+	(gr_line
+		(start 68.5 56)
+		(end 88.5 56)
 		(stroke
 			(width 0.15)
@@
 		(layer "Edge.Cuts")
 	)
-	(gr_line
-		(start 64 56)
-		(end 88 56)
+	(gr_arc
+		(start 66 58.5)
+		(mid 66.732233 56.732233)
+		(end 68.5 56)
 		(stroke
 			(width 0.15)
@@
 		(layer "Edge.Cuts")
 	)
-	(gr_circle
-		(center 64 63)
-		(end 65.414 63)
-		(stroke
-			(width 0.15)
-			(type solid)
-		)
-		(fill no)
-		(layer "Edge.Cuts")
-	)
 	(gr_arc
-		(start 61 59)
-		(mid 61.87868 56.87868)
-		(end 64 56)
+		(start 69 66)
+		(mid 66.87868 65.12132)
+		(end 66 63)
 		(stroke
 			(width 0.15)
@@
 		(layer "Edge.Cuts")
 	)
-	(gr_arc
-		(start 64 66)
-		(mid 61.87868 65.12132)
-		(end 61 63)
+	(gr_line
+		(start 88.5 66)
+		(end 69 66)
 		(stroke
 			(width 0.15)
@@
 	)
 	(gr_line
-		(start 88 66)
-		(end 64 66)
-		(stroke
-			(width 0.15)
-			(type default)
-		)
-		(layer "Edge.Cuts")
-	)
-	(gr_line
-		(start 91 59)
-		(end 91 63)
+		(start 91 58.5)
+		(end 91 63.5)
 		(stroke
 			(width 0.15)
@@
 	)
 	(gr_text "AS5600-Slim\n\n\n\nTanmayChhatbar"
-		(at 78 64.75 0)
+		(at 73 64.75 0)
 		(layer "B.SilkS")
 		(effects
@@
 				(thickness 0.153)
 			)
-			(justify left bottom mirror)
+			(justify bottom mirror)
 		)
 	)
@@
 		(net 1)
 	)
-	(segment
-		(start 71.4 64.6)
-		(end 84.86 64.6)
-		(width 0.5)
-		(layer "F.Cu")
-		(net 1)
-	)
 	(via
 		(at 68.5 62.5)
@@
 	)
 	(via
-		(at 71.4 64.6)
+		(at 84.86 64.6)
 		(size 0.25)
 		(drill 0.15)
@@
 	)
 	(segment
-		(start 71.4 64.6)
+		(start 84.86 64.6)
 		(end 69.6 64.6)
 		(width 0.5)
@@
 	)
 	(segment
+		(start 69.135 60.365)
+		(end 67.95 61.55)
+		(width 0.5)
+		(layer "F.Cu")
+		(net 5)
+	)
+	(segment
+		(start 80.190625 59.809375)
+		(end 79.6 60.4)
+		(width 0.5)
+		(layer "F.Cu")
+		(net 5)
+	)
+	(segment
 		(start 70.625 57.875)
 		(end 69.8625 58.6375)
@@
 	)
 	(segment
-		(start 80.190625 59.809375)
-		(end 79.6 60.4)
-		(width 0.5)
-		(layer "F.Cu")
-		(net 5)
-	)
-	(segment
 		(start 89 60.46)
 		(end 89 60)
@@
 	)
 	(segment
-		(start 67.855 59.095)
-		(end 67.5 59.45)
+		(start 67.95 61.55)
+		(end 67.5 61.55)
+		(width 0.5)
+		(layer "F.Cu")
+		(net 5)
+	)
+	(segment
+		(start 79.4625 60.6375)
+		(end 79.4625 62.5375)
+		(width 0.5)
+		(layer "F.Cu")
+		(net 5)
+	)
+	(segment
+		(start 89 60)
+		(end 87.5 58.5)
+		(width 0.5)
+		(layer "F.Cu")
+		(net 5)
+	)
+	(segment
+		(start 69.9 60.3275)
+		(end 69.8625 60.365)
+		(width 0.5)
+		(layer "F.Cu")
+		(net 5)
+	)
+	(segment
+		(start 79.425 60.6)
+		(end 79.4625 60.6375)
+		(width 0.5)
+		(layer "F.Cu")
+		(net 5)
+	)
+	(segment
+		(start 69.9 59.145)
+		(end 69.9 60.3275)
 		(width 0.5)
 		(layer "F.Cu")
@@
 	)
 	(segment
-		(start 79.4625 60.6375)
-		(end 79.4625 62.5375)
-		(width 0.5)
-		(layer "F.Cu")
-		(net 5)
-	)
-	(segment
-		(start 68.685 60.365)
-		(end 67.5 61.55)
-		(width 0.5)
-		(layer "F.Cu")
-		(net 5)
-	)
-	(segment
-		(start 89 60)
-		(end 87.5 58.5)
-		(width 0.5)
-		(layer "F.Cu")
-		(net 5)
-	)
-	(segment
-		(start 69.9 60.3275)
-		(end 69.8625 60.365)
-		(width 0.5)
-		(layer "F.Cu")
-		(net 5)
-	)
-	(segment
-		(start 79.425 60.6)
-		(end 79.4625 60.6375)
-		(width 0.5)
-		(layer "F.Cu")
-		(net 5)
-	)
-	(segment
-		(start 69.9 59.145)
-		(end 69.9 60.3275)
-		(width 0.5)
-		(layer "F.Cu")
-		(net 5)
-	)
-	(segment
-		(start 69.8625 60.545)
-		(end 69.6825 60.365)
-		(width 0.5)
-		(layer "F.Cu")
-		(net 5)
-	)
-	(segment
 		(start 69.8625 59.095)
-		(end 67.855 59.095)
+		(end 68.305 59.095)
+		(width 0.5)
+		(layer "F.Cu")
+		(net 5)
+	)
+	(segment
+		(start 69.6825 60.365)
+		(end 69.135 60.365)
+		(width 0.5)
+		(layer "F.Cu")
+		(net 5)
+	)
+	(segment
+		(start 68.305 59.095)
+		(end 67.5 59.9)
 		(width 0.5)
 		(layer "F.Cu")
@@
 		(start 79.4625 62.5375)
 		(end 79.4 62.6)
-		(width 0.5)
-		(layer "F.Cu")
-		(net 5)
-	)
-	(segment
-		(start 69.6825 60.365)
-		(end 68.685 60.365)
 		(width 0.5)
 		(layer "F.Cu")
@@
 	)
 	(segment
-		(start 74.25 63.75)
+		(start 67.5 64.5)
+		(end 68 65)
+		(width 0.5)
+		(layer "F.Cu")
+		(net 6)
+	)
+	(segment
+		(start 75.095 62.905)
+		(end 75.15 62.905)
+		(width 0.5)
+		(layer "F.Cu")
+		(net 6)
+	)
+	(segment
+		(start 75 63)
 		(end 75.095 62.905)
+		(width 0.5)
+		(layer "F.Cu")
+		(net 6)
+	)
+	(segment
+		(start 75 64)
+		(end 75 63)
 		(width 0.5)
 		(layer "F.Cu")
@@
 	)
 	(segment
-		(start 75.095 62.905)
-		(end 75.15 62.905)
+		(start 67.5 63.45)
+		(end 67.5 64.5)
 		(width 0.5)
 		(layer "F.Cu")
@@
 	)
 	(via
-		(at 67.4 64.5)
+		(at 68 65)
 		(size 0.25)
 		(drill 0.15)
@@
 	)
 	(via
-		(at 67.4 56.6)
+		(at 68 56.6)
 		(size 0.25)
 		(drill 0.15)
